Commit message: add urdf

File: ros2_robot_ws/src/moretea_description/urdf/moretea.urdf.xacro (robot description, xacro)
@@ -3,22 +3,15 @@
   <link name="base_footprint"/>
   <link name="base_link">
-    <inertial>
-      <origin xyz="0 0 0.04" rpy="0.0 0.25 0.3" />
-      <mass value="8.2573504e-01"/>
-      <inertia ixx="2.2124416e-02" ixy="-1.2294101e-04" ixz="3.4938785e-04"
-               iyy="2.1193702e-02" iyz="-5.0120904e-05"
-               izz="2.0064271e-02" />
-    </inertial>
     <visual>
-      <origin xyz="0 0 0" rpy="0 0 0" />
+      <origin xyz="-0.0925 0.0939 0.058" rpy="0 0 -1.5707963268"/>
       <geometry>
-        <mesh filename="package://moretea_description/meshes/base_link.STL" />
+        <mesh filename="package://moretea_description/meshes/base_link.stl" scale="0.001 0.001 0.001"/>
       </geometry>
-      <material name="black"/>
+      <material name="orange"/>
     </visual>
     <collision>
-      <origin xyz="0 0 0" rpy="0 0 0" />
+      <origin xyz="-0.0925 0.0939 0.058" rpy="0 0 -1.5707963268"/>
       <geometry>
-        <mesh filename="package://moretea_description/meshes/base_link.STL" />
+        <mesh filename="package://moretea_description/meshes/base_link.stl" scale="0.001 0.001 0.001"/>
       </geometry>
     </collision>
@@ -27,23 +20,16 @@
     <parent link="base_footprint"/>
     <child link="base_link" />
-    <origin xyz="0 0 0.033" rpy="0 0 0"/>
+    <origin xyz="0 0 0" rpy="0 0 0"/>
   </joint>
-  <link name="wheel_right_link">
-    <inertial>
-      <origin xyz="0 -0.014 0" rpy="0 0 0" />
-      <mass value="0.0530086090966721" />
-      <inertia ixx="1.88176298336665E-05" ixy="-4.8444933029987E-10" ixz="1.88163708851143E-08"
-               iyy="3.11510738647764E-05" iyz="-6.93560663069607E-11"
-               izz="1.8801969558182E-05" />
-    </inertial>
+  <link name="wheel_right_link_1">
     <visual>
-      <origin xyz="0 0 0" rpy="1.57 0 0" />
+      <origin xyz="0.03 -0.045 -0.029" rpy="0 0 1.5707963268"/>
       <geometry>
-        <mesh filename="package://moretea_description/meshes/wheel_right_link.STL" />
+        <mesh filename="package://moretea_description/meshes/mecanum_wheel.stl" scale="0.001 0.001 0.001"/>
       </geometry>
       <material name="blue"/>
     </visual>
     <collision>
-      <origin xyz="0 -0.015 0" rpy="1.57 0 0" />
+      <origin xyz="0.03 -0.045 -0.029" rpy="0 0 1.5707963268"/>
       <geometry>
         <sphere radius="0.033"/>
@@ -51,28 +37,20 @@
     </collision>
   </link>
-  <joint name="wheel_right_joint" type="continuous">
-    <origin xyz="0 -0.0701101849418637 0" rpy="0 0 0" />
+  <joint name="wheel_right_joint_1" type="continuous">
+    <origin xyz="0.0605 -0.07 0.029" rpy="0 0 0" />
     <parent link="base_link" />
-    <child link="wheel_right_link" />
+    <child link="wheel_right_link_1" />
     <axis xyz="0 1 0" />
   </joint>
-  <link
-    name="wheel_left_link">
-    <inertial>
-      <origin xyz="0 0.014 0" rpy="0 0 0" />
-      <mass value="0.0530086043217644" />
-      <inertia ixx="1.8792911368909E-05"  ixy="3.31256392204584E-10" ixz="-1.14082001662767E-08"
-               iyy="3.11510738759073E-05" iyz="-3.60499245082192E-10"
-               izz="1.88266886146847E-05" />
-    </inertial>
+  <link name="wheel_right_link_2">
     <visual>
-      <origin xyz="0 0 0" rpy="-1.57 0 0" />
+      <origin xyz="0.03 -0.045 -0.029" rpy="0 0 1.5707963268"/>
       <geometry>
-        <mesh filename="package://moretea_description/meshes/wheel_left_link.STL" />
+        <mesh filename="package://moretea_description/meshes/mecanum_wheel.stl" scale="0.001 0.001 0.001"/>
       </geometry>
       <material name="blue"/>
     </visual>
     <collision>
-      <origin xyz="0 0.015 0" rpy="-1.57 0 0" />
+      <origin xyz="0.03 -0.045 -0.029" rpy="0 0 1.5707963268"/>
       <geometry>
         <sphere radius="0.033"/>
@@ -80,65 +58,51 @@
     </collision>
   </link>
-  <joint name="wheel_left_joint" type="continuous">
-    <origin xyz="0 0.0701101849418642 0" rpy="0 0 0" />
+  <joint name="wheel_right_joint_2" type="continuous">
+    <origin xyz="-0.0605 -0.07 0.029" rpy="0 0 0" />
     <parent link="base_link" />
-    <child link="wheel_left_link" />
+    <child link="wheel_right_link_2" />
     <axis xyz="0 1 0" />
   </joint>
-  <link name="caster_front_link">
-    <inertial>
-      <origin xyz="3.89968128948481E-07 2.40073004698083E-07 0.00219173397061506" rpy="0 0 0" />
-      <mass value="1.44379265037903E-06" />
-      <inertia ixx="7.23075276010246E-11" ixy="-6.10956883467859E-16" ixz="2.22849693525031E-15"
-               iyy="3.8713793085917E-11"  iyz="2.93909858781952E-15"
-               izz="1.00967486676306E-10" />
-    </inertial>
+  <link name="wheel_left_link_1">
     <visual>
-      <origin xyz="0 0 0" rpy="0 0 0" />
+      <origin xyz="-0.03 0.045 -0.029" rpy="0 0 -1.5707963268"/>
       <geometry>
-        <mesh filename="package://moretea_description/meshes/caster_front_link.STL" />
+        <mesh filename="package://moretea_description/meshes/mecanum_wheel.stl" scale="0.001 0.001 0.001"/>
       </geometry>
-      <material name="silver"/>
+      <material name="blue"/>
     </visual>
     <collision>
-      <origin xyz="0 0 0" rpy="0 0 0" />
+      <origin xyz="-0.03 0.045 -0.029" rpy="0 0 -1.5707963268"/>
       <geometry>
-        <sphere radius="0.005"/>
+        <sphere radius="0.033"/>
       </geometry>
     </collision>
   </link>
-  <joint name="caster_front_joint" type="fixed">
-    <origin xyz="0.04755 0 -0.0275" rpy="0 0 0" />
+  <joint name="wheel_left_joint_1" type="continuous">
+    <origin xyz="0.0605 0.07 0.029" rpy="0 0 0" />
     <parent link="base_link" />
-    <child link="caster_front_link" />
-    <axis xyz="0 0 0" />
+    <child link="wheel_left_link_1" />
+    <axis xyz="0 1 0" />
   </joint>
-  <link name="caster_rear_link">
-    <inertial>
-      <origin xyz="3.8996812895542E-07 2.40073004698083E-07 0.00219173397061509" rpy="0 0 0" />
-      <mass value="1.44379265037902E-06" />
-      <inertia ixx="7.23075276010246E-11" ixy="-6.10956872363424E-16" ixz="2.22849693527207E-15"
-               iyy="3.87137930859167E-11" iyz="2.939098587861E-15"
-               izz="1.00967486676306E-10" />
-    </inertial>
+  <link name="wheel_left_link_2">
     <visual>
-      <origin xyz="0 0 0" rpy="0 0 0" />
+      <origin xyz="-0.03 0.045 -0.029" rpy="0 0 -1.5707963268"/>
       <geometry>
-        <mesh filename="package://moretea_description/meshes/caster_rear_link.STL" />
+        <mesh filename="package://moretea_description/meshes/mecanum_wheel.stl" scale="0.001 0.001 0.001"/>
       </geometry>
-      <material name="silver"/>
+      <material name="blue"/>
     </visual>
     <collision>
-      <origin xyz="0 0 0" rpy="0 0 0" />
+      <origin xyz="-0.03 0.045 -0.029" rpy="0 0 -1.5707963268"/>
       <geometry>
-        <sphere radius="0.005"/>
+        <sphere radius="0.033"/>
       </geometry>
     </collision>
   </link>
-  <joint name="caster_rear_joint" type="fixed">
-    <origin xyz="-0.04755 0 -0.0275" rpy="0 0 0" />
+  <joint name="wheel_left_joint_2" type="continuous">
+    <origin xyz="-0.0605 0.07 0.029" rpy="0 0 0" />
     <parent link="base_link" />
-    <child link="caster_rear_link" />
-    <axis xyz="0 0 0" />
+    <child link="wheel_left_link_2" />
+    <axis xyz="0 1 0" />
   </joint>
   <link name="imu_link">
@@ -151,19 +115,19 @@
     </inertial>
     <visual>
-      <origin xyz="0 0 0" rpy="0 0 0" />
+      <origin xyz="-0.0075 -0.01 0" rpy="0 0 0" />
       <geometry>
-        <mesh filename="package://moretea_description/meshes/imu_link.STL" />
+        <mesh filename="package://moretea_description/meshes/imu_link.STL" scale="0.001 0.001 0.001"/>
       </geometry>
       <material name="blue"/>
     </visual>
     <collision>
-      <origin xyz="0 0 0" rpy="0 0 0" />
+      <origin xyz="-0.0075 -0.01 0" rpy="0 0 0" />
       <geometry>
-        <mesh filename="package://moretea_description/meshes/imu_link.STL" />
+        <mesh filename="package://moretea_description/meshes/imu_link.STL" scale="0.001 0.001 0.001"/>
       </geometry>
     </collision>
   </link>
   <joint name="imu_joint" type="fixed">
-    <origin xyz="0 0 0.0698986241758014" rpy="0 0 0" />
+    <origin xyz="0 0 0.029" rpy="0 0 0" />
     <parent link="base_link" />
     <child link="imu_link" />
@@ -182,3 +146,6 @@
     <color rgba="0.3 0.3 0.3 1"/>
   </material>
+  <material name="orange">
+  <color rgba="${255/255} ${108/255} ${10/255} 1.0"/>
+  </material>
 </robot>

Commit message: update moretea_controller

File: ros2_robot_ws/src/moretea_description/urdf/moretea.urdf.xacro (robot description, xacro)
@@ -1,6 +1,17 @@
 <?xml version="1.0"?>
 <robot name="moretea" xmlns:xacro="http://ros.org/wiki/xacro">
+  <!-- Include Gazebo Parameters -->
+  <xacro:include filename="$(find moretea_description)/urdf/moretea_gazebo.xacro"/>
+  <!-- ROS 2 Control -->
+  <xacro:include filename="$(find moretea_description)/urdf/moretea_ros2_control.xacro"/>
   <link name="base_footprint"/>
   <link name="base_link">
+    <inertial>
+      <origin xyz="0 0 0.04" rpy="0.0 0.25 0.3" />
+      <mass value="8.2573504e-01"/>
+      <inertia ixx="2.2124416e-02" ixy="-1.2294101e-04" ixz="3.4938785e-04"
+               iyy="2.1193702e-02" iyz="-5.0120904e-05"
+               izz="2.0064271e-02" />
+    </inertial>
     <visual>
       <origin xyz="-0.0925 0.0939 0.058" rpy="0 0 -1.5707963268"/>
@@ -23,4 +34,11 @@
   </joint>
   <link name="wheel_right_link_1">
+    <inertial>
+      <origin xyz="0 -0.014 0" rpy="0 0 0" />
+      <mass value="0.0530086090966721" />
+      <inertia ixx="1.88176298336665E-05" ixy="-4.8444933029987E-10" ixz="1.88163708851143E-08"
+               iyy="3.11510738647764E-05" iyz="-6.93560663069607E-11"
+               izz="1.8801969558182E-05" />
+    </inertial>
     <visual>
       <origin xyz="0.03 -0.045 -0.029" rpy="0 0 1.5707963268"/>
@@ -31,7 +49,7 @@
     </visual>
     <collision>
-      <origin xyz="0.03 -0.045 -0.029" rpy="0 0 1.5707963268"/>
+      <origin xyz="0 -0.025 0" rpy="0 0 1.5707963268"/>
       <geometry>
-        <sphere radius="0.033"/>
+        <sphere radius="0.029"/>
       </geometry>
     </collision>
@@ -44,4 +62,11 @@
   </joint>
   <link name="wheel_right_link_2">
+    <inertial>
+      <origin xyz="0 -0.014 0" rpy="0 0 0"/>
+      <mass value="0.0530086090966721"/>
+      <inertia ixx="1.88176298336665E-05" ixy="-4.8444933029987E-10" ixz="1.88163708851143E-08"
+               iyy="3.11510738647764E-05" iyz="-6.93560663069607E-11"
+               izz="1.8801969558182E-05"/>
+    </inertial>
     <visual>
       <origin xyz="0.03 -0.045 -0.029" rpy="0 0 1.5707963268"/>
@@ -52,7 +77,7 @@
     </visual>
     <collision>
-      <origin xyz="0.03 -0.045 -0.029" rpy="0 0 1.5707963268"/>
+      <origin xyz="0 -0.025 0" rpy="0 0 1.5707963268"/>
       <geometry>
-        <sphere radius="0.033"/>
+        <sphere radius="0.029"/>
       </geometry>
     </collision>
@@ -65,4 +90,11 @@
   </joint>
   <link name="wheel_left_link_1">
+    <inertial>
+      <origin xyz="0 0.014 0" rpy="0 0 0" />
+      <mass value="0.0530086043217644" />
+      <inertia ixx="1.8792911368909E-05"  ixy="3.31256392204584E-10" ixz="-1.14082001662767E-08"
+               iyy="3.11510738759073E-05" iyz="-3.60499245082192E-10"
+               izz="1.88266886146847E-05" />
+    </inertial>
     <visual>
       <origin xyz="-0.03 0.045 -0.029" rpy="0 0 -1.5707963268"/>
@@ -73,7 +105,7 @@
     </visual>
     <collision>
-      <origin xyz="-0.03 0.045 -0.029" rpy="0 0 -1.5707963268"/>
+      <origin xyz="0 0.025 0" rpy="0 0 -1.5707963268"/>
       <geometry>
-        <sphere radius="0.033"/>
+        <sphere radius="0.029"/>
       </geometry>
     </collision>
@@ -86,4 +118,11 @@
   </joint>
   <link name="wheel_left_link_2">
+    <inertial>
+      <origin xyz="0 0.014 0" rpy="0 0 0" />
+      <mass value="0.0530086043217644" />
+      <inertia ixx="1.8792911368909E-05"  ixy="3.31256392204584E-10" ixz="-1.14082001662767E-08"
+               iyy="3.11510738759073E-05" iyz="-3.60499245082192E-10"
+               izz="1.88266886146847E-05" />
+    </inertial>
     <visual>
       <origin xyz="-0.03 0.045 -0.029" rpy="0 0 -1.5707963268"/>
@@ -94,7 +133,7 @@
     </visual>
     <collision>
-      <origin xyz="-0.03 0.045 -0.029" rpy="0 0 -1.5707963268"/>
+      <origin xyz="0 0.025 0" rpy="0 0 -1.5707963268"/>
       <geometry>
-        <sphere radius="0.033"/>
+        <sphere radius="0.029"/>
       </geometry>
     </collision>

Commit message: update

File: ros2_robot_ws/src/moretea_description/urdf/moretea.urdf.xacro (robot description, xacro)
@@ -1,4 +1,5 @@
 <?xml version="1.0"?>
 <robot name="moretea" xmlns:xacro="http://ros.org/wiki/xacro">
+  <xacro:arg name="is_ignition" default="true"/>
   <!-- Include Gazebo Parameters -->
   <xacro:include filename="$(find moretea_description)/urdf/moretea_gazebo.xacro"/>
@@ -8,6 +9,6 @@
   <link name="base_link">
     <inertial>
-      <origin xyz="0 0 0.04" rpy="0.0 0.25 0.3" />
-      <mass value="8.2573504e-01"/>
+      <origin xyz="0 0 0.04" rpy="0 0 0" />
+      <mass value="10"/>
       <inertia ixx="2.2124416e-02" ixy="-1.2294101e-04" ixz="3.4938785e-04"
                iyy="2.1193702e-02" iyz="-5.0120904e-05"
@@ -36,8 +37,6 @@
     <inertial>
       <origin xyz="0 -0.014 0" rpy="0 0 0" />
-      <mass value="0.0530086090966721" />
-      <inertia ixx="1.88176298336665E-05" ixy="-4.8444933029987E-10" ixz="1.88163708851143E-08"
-               iyy="3.11510738647764E-05" iyz="-6.93560663069607E-11"
-               izz="1.8801969558182E-05" />
+      <mass value="0.5" />
+      <inertia ixx="0.001" ixy="0" ixz="0" iyy="0.001" iyz="0" izz="0.001" />
     </inertial>
     <visual>
@@ -64,8 +63,6 @@
     <inertial>
       <origin xyz="0 -0.014 0" rpy="0 0 0"/>
-      <mass value="0.0530086090966721"/>
-      <inertia ixx="1.88176298336665E-05" ixy="-4.8444933029987E-10" ixz="1.88163708851143E-08"
-               iyy="3.11510738647764E-05" iyz="-6.93560663069607E-11"
-               izz="1.8801969558182E-05"/>
+      <mass value="0.5" />
+      <inertia ixx="0.001" ixy="0" ixz="0" iyy="0.001" iyz="0" izz="0.001"/>
     </inertial>
     <visual>
@@ -92,8 +89,6 @@
     <inertial>
       <origin xyz="0 0.014 0" rpy="0 0 0" />
-      <mass value="0.0530086043217644" />
-      <inertia ixx="1.8792911368909E-05"  ixy="3.31256392204584E-10" ixz="-1.14082001662767E-08"
-               iyy="3.11510738759073E-05" iyz="-3.60499245082192E-10"
-               izz="1.88266886146847E-05" />
+      <mass value="0.5" />
+      <inertia ixx="0.001" ixy="0" ixz="0" iyy="0.001" iyz="0" izz="0.001" />
     </inertial>
     <visual>
@@ -120,8 +115,6 @@
     <inertial>
       <origin xyz="0 0.014 0" rpy="0 0 0" />
-      <mass value="0.0530086043217644" />
-      <inertia ixx="1.8792911368909E-05"  ixy="3.31256392204584E-10" ixz="-1.14082001662767E-08"
-               iyy="3.11510738759073E-05" iyz="-3.60499245082192E-10"
-               izz="1.88266886146847E-05" />
+      <mass value="0.5" />
+      <inertia ixx="0.001" ixy="0" ixz="0" iyy="0.001" iyz="0" izz="0.001" />
     </inertial>
     <visual>

File: ros2_robot_ws/src/moretea_description/urdf/moretea_gazebo.xacro (robot description, xacro)
@@ -1,40 +1,41 @@
 <?xml version="1.0"?>
 <robot name="moretea" xmlns:xacro="http://ros.org/wiki/xacro">
-  <!-- Wheels -->
+  <!-- Mecanum Wheels Friction Configuration -->
+  <!-- Standard "O" configuration: FL & RR have same roller angle, FR & RL have same roller angle -->
+  <!-- Front Left (wheel_left_link_1) - roller angle 45° -->
   <gazebo reference="wheel_left_link_1">
-    <mu1>1000000000000000.0</mu1>
-    <mu2>1000000000000000.0</mu2>
-    <kp>1000000000000.0</kp>
-    <kd>10.0</kd>
+    <mu1>1.0</mu1>
+    <mu2>0.0</mu2>
+    <kp>1000000.0</kp>
+    <kd>100.0</kd>
     <minDepth>0.001</minDepth>
-    <maxVel>0.1</maxVel>
-    <fdir1>1 0 0</fdir1>
+    <fdir1>1 1 0</fdir1>
   </gazebo>
+  <!-- Rear Left (wheel_left_link_2) - roller angle -45° -->
   <gazebo reference="wheel_left_link_2">
-    <mu1>1000000000000000.0</mu1>
-    <mu2>1000000000000000.0</mu2>
-    <kp>1000000000000.0</kp>
-    <kd>10.0</kd>
+    <mu1>1.0</mu1>
+    <mu2>0.0</mu2>
+    <kp>1000000.0</kp>
+    <kd>100.0</kd>
     <minDepth>0.001</minDepth>
-    <maxVel>0.1</maxVel>
-    <fdir1>1 0 0</fdir1>
+    <fdir1>1 -1 0</fdir1>
   </gazebo>
+  <!-- Front Right (wheel_right_link_1) - roller angle -45° -->
   <gazebo reference="wheel_right_link_1">
-    <mu1>1000000000000000.0</mu1>
-    <mu2>1000000000000000.0</mu2>
-    <kp>1000000000000.0</kp>
-    <kd>10.0</kd>
+    <mu1>1.0</mu1>
+    <mu2>0.0</mu2>
+    <kp>1000000.0</kp>
+    <kd>100.0</kd>
     <minDepth>0.001</minDepth>
-    <maxVel>0.1</maxVel>
-    <fdir1>1 0 0</fdir1>
+    <fdir1>1 -1 0</fdir1>
   </gazebo>
+  <!-- Rear Right (wheel_right_link_2) - roller angle 45° -->
   <gazebo reference="wheel_right_link_2">
-    <mu1>1000000000000000.0</mu1>
-    <mu2>1000000000000000.0</mu2>
-    <kp>1000000000000.0</kp>
-    <kd>10.0</kd>
+    <mu1>1.0</mu1>
+    <mu2>0.0</mu2>
+    <kp>1000000.0</kp>
+    <kd>100.0</kd>
     <minDepth>0.001</minDepth>
-    <maxVel>0.1</maxVel>
-    <fdir1>1 0 0</fdir1>
+    <fdir1>1 1 0</fdir1>
   </gazebo>
   <!-- ROS 2 Control -->
