Commit message: update

File: ros2_robot_ws/src/moretea_description/urdf/moretea.urdf.xacro (robot description, xacro)
@@ -9,5 +9,5 @@
   <link name="base_link">
     <inertial>
-      <origin xyz="0 0 0.04" rpy="0 0 0" />
+      <origin xyz="0 0 0.12" rpy="0 0 0" />
       <mass value="10"/>
       <inertia ixx="2.2124416e-02" ixy="-1.2294101e-04" ixz="3.4938785e-04"
@@ -16,5 +16,5 @@
     </inertial>
     <visual>
-      <origin xyz="-0.0925 0.0939 0.058" rpy="0 0 -1.5707963268"/>
+      <origin xyz="0 0 0.12" rpy="3.14159 0 -1.5707963268"/>
       <geometry>
         <mesh filename="package://moretea_description/meshes/base_link.stl" scale="0.001 0.001 0.001"/>
@@ -23,5 +23,5 @@
     </visual>
     <collision>
-      <origin xyz="-0.0925 0.0939 0.058" rpy="0 0 -1.5707963268"/>
+      <origin xyz="0 0 0.12" rpy="3.14159 0 -1.5707963268"/>
       <geometry>
         <mesh filename="package://moretea_description/meshes/base_link.stl" scale="0.001 0.001 0.001"/>
@@ -36,10 +36,12 @@
   <link name="wheel_right_link_1">
     <inertial>
-      <origin xyz="0 -0.014 0" rpy="0 0 0" />
+      <origin xyz="0 -0.023 0" rpy="0 0 0" />
       <mass value="0.5" />
-      <inertia ixx="0.001" ixy="0" ixz="0" iyy="0.001" iyz="0" izz="0.001" />
+      <inertia ixx="0.000195" ixy="0" ixz="0"
+               iyy="0.000215" iyz="0"
+               izz="0.000195" />
     </inertial>
     <visual>
-      <origin xyz="0.03 -0.045 -0.029" rpy="0 0 1.5707963268"/>
+      <origin xyz="0.029315 -0.04132 -0.029315" rpy="0 0 1.5707963268"/>
       <geometry>
         <mesh filename="package://moretea_description/meshes/mecanum_wheel.stl" scale="0.001 0.001 0.001"/>
@@ -48,24 +50,27 @@
     </visual>
     <collision>
-      <origin xyz="0 -0.025 0" rpy="0 0 1.5707963268"/>
+      <origin xyz="0 -0.023 0" rpy="1.5707963268 0 0"/>
       <geometry>
-        <sphere radius="0.029"/>
+        <cylinder radius="0.029315" length="0.046"/>
       </geometry>
     </collision>
   </link>
   <joint name="wheel_right_joint_1" type="continuous">
-    <origin xyz="0.0605 -0.07 0.029" rpy="0 0 0" />
+    <origin xyz="0.105 -0.08 0.029315" rpy="0 0 0" />
     <parent link="base_link" />
     <child link="wheel_right_link_1" />
     <axis xyz="0 1 0" />
+    <dynamics damping="0.1"/>
   </joint>
   <link name="wheel_right_link_2">
     <inertial>
-      <origin xyz="0 -0.014 0" rpy="0 0 0"/>
+      <origin xyz="0 -0.023 0" rpy="0 0 0"/>
       <mass value="0.5" />
-      <inertia ixx="0.001" ixy="0" ixz="0" iyy="0.001" iyz="0" izz="0.001"/>
+      <inertia ixx="0.000195" ixy="0" ixz="0"
+               iyy="0.000215" iyz="0"
+               izz="0.000195" />
     </inertial>
     <visual>
-      <origin xyz="0.03 -0.045 -0.029" rpy="0 0 1.5707963268"/>
+      <origin xyz="0.029315 -0.04132 -0.029315" rpy="0 0 1.5707963268"/>
       <geometry>
         <mesh filename="package://moretea_description/meshes/mecanum_wheel.stl" scale="0.001 0.001 0.001"/>
@@ -74,24 +79,27 @@
     </visual>
     <collision>
-      <origin xyz="0 -0.025 0" rpy="0 0 1.5707963268"/>
+      <origin xyz="0 -0.023 0" rpy="1.5707963268 0 0"/>
       <geometry>
-        <sphere radius="0.029"/>
+        <cylinder radius="0.029315" length="0.046"/>
       </geometry>
     </collision>
   </link>
   <joint name="wheel_right_joint_2" type="continuous">
-    <origin xyz="-0.0605 -0.07 0.029" rpy="0 0 0" />
+    <origin xyz="-0.105 -0.08 0.029315" rpy="0 0 0" />
     <parent link="base_link" />
     <child link="wheel_right_link_2" />
     <axis xyz="0 1 0" />
+    <dynamics damping="0.1"/>
   </joint>
   <link name="wheel_left_link_1">
     <inertial>
-      <origin xyz="0 0.014 0" rpy="0 0 0" />
+      <origin xyz="0 0.023 0" rpy="0 0 0" />
       <mass value="0.5" />
-      <inertia ixx="0.001" ixy="0" ixz="0" iyy="0.001" iyz="0" izz="0.001" />
+      <inertia ixx="0.000195" ixy="0" ixz="0"
+               iyy="0.000215" iyz="0"
+               izz="0.000195" />
     </inertial>
     <visual>
-      <origin xyz="-0.03 0.045 -0.029" rpy="0 0 -1.5707963268"/>
+      <origin xyz="-0.029315 0.04132 -0.029315" rpy="0 0 -1.5707963268"/>
       <geometry>
         <mesh filename="package://moretea_description/meshes/mecanum_wheel.stl" scale="0.001 0.001 0.001"/>
@@ -100,24 +108,27 @@
     </visual>
     <collision>
-      <origin xyz="0 0.025 0" rpy="0 0 -1.5707963268"/>
+      <origin xyz="0 0.023 0" rpy="1.5707963268 0 0"/>
       <geometry>
-        <sphere radius="0.029"/>
+        <cylinder radius="0.029315" length="0.046"/>
       </geometry>
     </collision>
   </link>
   <joint name="wheel_left_joint_1" type="continuous">
-    <origin xyz="0.0605 0.07 0.029" rpy="0 0 0" />
+    <origin xyz="0.105 0.08 0.029315" rpy="0 0 0" />
     <parent link="base_link" />
     <child link="wheel_left_link_1" />
     <axis xyz="0 1 0" />
+    <dynamics damping="0.1"/>
   </joint>
   <link name="wheel_left_link_2">
     <inertial>
-      <origin xyz="0 0.014 0" rpy="0 0 0" />
+      <origin xyz="0 0.023 0" rpy="0 0 0" />
       <mass value="0.5" />
-      <inertia ixx="0.001" ixy="0" ixz="0" iyy="0.001" iyz="0" izz="0.001" />
+      <inertia ixx="0.000195" ixy="0" ixz="0"
+               iyy="0.000215" iyz="0"
+               izz="0.000195" />
     </inertial>
     <visual>
-      <origin xyz="-0.03 0.045 -0.029" rpy="0 0 -1.5707963268"/>
+      <origin xyz="-0.029315 0.04132 -0.029315" rpy="0 0 -1.5707963268"/>
       <geometry>
         <mesh filename="package://moretea_description/meshes/mecanum_wheel.stl" scale="0.001 0.001 0.001"/>
@@ -126,15 +137,16 @@
     </visual>
     <collision>
-      <origin xyz="0 0.025 0" rpy="0 0 -1.5707963268"/>
+      <origin xyz="0 0.023 0" rpy="1.5707963268 0 0"/>
       <geometry>
-        <sphere radius="0.029"/>
+        <cylinder radius="0.029315" length="0.046"/>
       </geometry>
     </collision>
   </link>
   <joint name="wheel_left_joint_2" type="continuous">
-    <origin xyz="-0.0605 0.07 0.029" rpy="0 0 0" />
+    <origin xyz="-0.105 0.08 0.029315" rpy="0 0 0" />
     <parent link="base_link" />
     <child link="wheel_left_link_2" />
     <axis xyz="0 1 0" />
+    <dynamics damping="0.1"/>
   </joint>
   <link name="imu_link">

File: ros2_robot_ws/src/moretea_description/urdf/moretea_gazebo.xacro (robot description, xacro)
@@ -3,8 +3,18 @@
   <!-- Mecanum Wheels Friction Configuration -->
   <!-- Standard "O" configuration: FL & RR have same roller angle, FR & RL have same roller angle -->
+  <!-- fdir1 is in WORLD frame, considering wheel positions and roller angles -->
   <!-- Front Left (wheel_left_link_1) - roller angle 45° -->
   <gazebo reference="wheel_left_link_1">
     <mu1>1.0</mu1>
-    <mu2>0.0</mu2>
+    <mu2>0.01</mu2>
+    <kp>1000000.0</kp>
+    <kd>100.0</kd>
+    <minDepth>0.001</minDepth>
+    <fdir1>1 -1 0</fdir1>
+  </gazebo>
+  <!-- Rear Left (wheel_left_link_2) - roller angle -45° -->
+  <gazebo reference="wheel_left_link_2">
+    <mu1>1.0</mu1>
+    <mu2>0.01</mu2>
     <kp>1000000.0</kp>
     <kd>100.0</kd>
@@ -12,30 +22,21 @@
     <fdir1>1 1 0</fdir1>
   </gazebo>
-  <!-- Rear Left (wheel_left_link_2) - roller angle -45° -->
-  <gazebo reference="wheel_left_link_2">
+  <!-- Front Right (wheel_right_link_1) - roller angle -45° -->
+  <gazebo reference="wheel_right_link_1">
     <mu1>1.0</mu1>
-    <mu2>0.0</mu2>
+    <mu2>0.01</mu2>
+    <kp>1000000.0</kp>
+    <kd>100.0</kd>
+    <minDepth>0.001</minDepth>
+    <fdir1>1 1 0</fdir1>
+  </gazebo>
+  <!-- Rear Right (wheel_right_link_2) - roller angle 45° -->
+  <gazebo reference="wheel_right_link_2">
+    <mu1>1.0</mu1>
+    <mu2>0.01</mu2>
     <kp>1000000.0</kp>
     <kd>100.0</kd>
     <minDepth>0.001</minDepth>
     <fdir1>1 -1 0</fdir1>
-  </gazebo>
-  <!-- Front Right (wheel_right_link_1) - roller angle -45° -->
-  <gazebo reference="wheel_right_link_1">
-    <mu1>1.0</mu1>
-    <mu2>0.0</mu2>
-    <kp>1000000.0</kp>
-    <kd>100.0</kd>
-    <minDepth>0.001</minDepth>
-    <fdir1>1 -1 0</fdir1>
-  </gazebo>
-  <!-- Rear Right (wheel_right_link_2) - roller angle 45° -->
-  <gazebo reference="wheel_right_link_2">
-    <mu1>1.0</mu1>
-    <mu2>0.0</mu2>
-    <kp>1000000.0</kp>
-    <kd>100.0</kd>
-    <minDepth>0.001</minDepth>
-    <fdir1>1 1 0</fdir1>
   </gazebo>
   <!-- ROS 2 Control -->

Commit message: update controller

File: ros2_robot_ws/src/moretea_description/urdf/moretea.urdf.xacro (robot description, xacro)
@@ -6,4 +6,6 @@
   <!-- ROS 2 Control -->
   <xacro:include filename="$(find moretea_description)/urdf/moretea_ros2_control.xacro"/>
+  <!-- Mecanum Wheel Properties -->
+  <xacro:include filename="$(find moretea_description)/urdf/mecanum_properties.urdf.xacro"/>
   <link name="base_footprint"/>
   <link name="base_link">
@@ -37,8 +39,8 @@
     <inertial>
       <origin xyz="0 -0.023 0" rpy="0 0 0" />
-      <mass value="0.5" />
-      <inertia ixx="0.000195" ixy="0" ixz="0"
-               iyy="0.000215" iyz="0"
-               izz="0.000195" />
+      <mass value="${wheel_mass}" />
+      <inertia ixx="${(2/5) * wheel_mass * (wheel_radius * wheel_radius)}" ixy="0" ixz="0"
+               iyy="${(2/5) * wheel_mass * (wheel_radius * wheel_radius)}" iyz="0"
+               izz="${(2/5) * wheel_mass * (wheel_radius * wheel_radius)}" />
     </inertial>
     <visual>
@@ -52,5 +54,5 @@
       <origin xyz="0 -0.023 0" rpy="1.5707963268 0 0"/>
       <geometry>
-        <cylinder radius="0.029315" length="0.046"/>
+        <cylinder radius="${wheel_radius}" length="${wheel_width}"/>
       </geometry>
     </collision>
@@ -66,8 +68,8 @@
     <inertial>
       <origin xyz="0 -0.023 0" rpy="0 0 0"/>
-      <mass value="0.5" />
-      <inertia ixx="0.000195" ixy="0" ixz="0"
-               iyy="0.000215" iyz="0"
-               izz="0.000195" />
+      <mass value="${wheel_mass}" />
+      <inertia ixx="${(2/5) * wheel_mass * (wheel_radius * wheel_radius)}" ixy="0" ixz="0"
+               iyy="${(2/5) * wheel_mass * (wheel_radius * wheel_radius)}" iyz="0"
+               izz="${(2/5) * wheel_mass * (wheel_radius * wheel_radius)}" />
     </inertial>
     <visual>
@@ -81,5 +83,5 @@
       <origin xyz="0 -0.023 0" rpy="1.5707963268 0 0"/>
       <geometry>
-        <cylinder radius="0.029315" length="0.046"/>
+        <cylinder radius="${wheel_radius}" length="${wheel_width}"/>
       </geometry>
     </collision>
@@ -95,8 +97,8 @@
     <inertial>
       <origin xyz="0 0.023 0" rpy="0 0 0" />
-      <mass value="0.5" />
-      <inertia ixx="0.000195" ixy="0" ixz="0"
-               iyy="0.000215" iyz="0"
-               izz="0.000195" />
+      <mass value="${wheel_mass}" />
+      <inertia ixx="${(2/5) * wheel_mass * (wheel_radius * wheel_radius)}" ixy="0" ixz="0"
+               iyy="${(2/5) * wheel_mass * (wheel_radius * wheel_radius)}" iyz="0"
+               izz="${(2/5) * wheel_mass * (wheel_radius * wheel_radius)}" />
     </inertial>
     <visual>
@@ -110,5 +112,5 @@
       <origin xyz="0 0.023 0" rpy="1.5707963268 0 0"/>
       <geometry>
-        <cylinder radius="0.029315" length="0.046"/>
+        <cylinder radius="${wheel_radius}" length="${wheel_width}"/>
       </geometry>
     </collision>
@@ -124,8 +126,8 @@
     <inertial>
       <origin xyz="0 0.023 0" rpy="0 0 0" />
-      <mass value="0.5" />
-      <inertia ixx="0.000195" ixy="0" ixz="0"
-               iyy="0.000215" iyz="0"
-               izz="0.000195" />
+      <mass value="${wheel_mass}" />
+      <inertia ixx="${(2/5) * wheel_mass * (wheel_radius * wheel_radius)}" ixy="0" ixz="0"
+               iyy="${(2/5) * wheel_mass * (wheel_radius * wheel_radius)}" iyz="0"
+               izz="${(2/5) * wheel_mass * (wheel_radius * wheel_radius)}" />
     </inertial>
     <visual>
@@ -139,5 +141,5 @@
       <origin xyz="0 0.023 0" rpy="1.5707963268 0 0"/>
       <geometry>
-        <cylinder radius="0.029315" length="0.046"/>
+        <cylinder radius="${wheel_radius}" length="${wheel_width}"/>
       </geometry>
     </collision>

File: ros2_robot_ws/src/moretea_description/urdf/moretea_gazebo.xacro (robot description, xacro)
@@ -6,37 +6,33 @@
   <!-- Front Left (wheel_left_link_1) - roller angle 45° -->
   <gazebo reference="wheel_left_link_1">
-    <mu1>1.0</mu1>
-    <mu2>0.01</mu2>
-    <kp>1000000.0</kp>
-    <kd>100.0</kd>
-    <minDepth>0.001</minDepth>
-    <fdir1>1 -1 0</fdir1>
+    <mu1>0.1</mu1>
+    <mu2>0.1</mu2>
+    <kp>200000.0</kp>
+    <kd>5000.0</kd>
+    <!-- <fdir1>1 -1 0</fdir1> -->
   </gazebo>
   <!-- Rear Left (wheel_left_link_2) - roller angle -45° -->
   <gazebo reference="wheel_left_link_2">
-    <mu1>1.0</mu1>
-    <mu2>0.01</mu2>
-    <kp>1000000.0</kp>
-    <kd>100.0</kd>
-    <minDepth>0.001</minDepth>
-    <fdir1>1 1 0</fdir1>
+    <mu1>0.0</mu1>
+    <mu2>0.0</mu2>
+    <kp>200000.0</kp>
+    <kd>5000.0</kd>
+    <!-- <fdir1>1 1 0</fdir1> -->
   </gazebo>
   <!-- Front Right (wheel_right_link_1) - roller angle -45° -->
   <gazebo reference="wheel_right_link_1">
-    <mu1>1.0</mu1>
-    <mu2>0.01</mu2>
-    <kp>1000000.0</kp>
-    <kd>100.0</kd>
-    <minDepth>0.001</minDepth>
-    <fdir1>1 1 0</fdir1>
+    <mu1>0.1</mu1>
+    <mu2>0.1</mu2>
+    <kp>200000.0</kp>
+    <kd>5000.0</kd>
+    <!-- <fdir1>1 1 0</fdir1> -->
   </gazebo>
   <!-- Rear Right (wheel_right_link_2) - roller angle 45° -->
   <gazebo reference="wheel_right_link_2">
-    <mu1>1.0</mu1>
-    <mu2>0.01</mu2>
-    <kp>1000000.0</kp>
-    <kd>100.0</kd>
-    <minDepth>0.001</minDepth>
-    <fdir1>1 -1 0</fdir1>
+    <mu1>0.0</mu1>
+    <mu2>0.0</mu2>
+    <kp>200000.0</kp>
+    <kd>5000.0</kd>
+    <!-- <fdir1>1 -1 0</fdir1> -->
   </gazebo>
   <!-- ROS 2 Control -->
